File: hardware/main-board/BoatHub.kicad_pcb (KiCad board)
At the start: 2 copper layers, 134.6 x 91.4 mm, 58 parts, among them J1 Conn_01x08_Socket (ADS breako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, J10 Conn_01x10_Socket (ADS1115 2), J11 ESP32-S3-N16R8-DevKit_01x22_S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, J12 Screw_Terminal_01x02 (Bilge d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, J14 Screw_Terminal_01x04 (DS18B F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, J15 Screw_Terminal_01x04 (DS18B B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, J16 Screw_Terminal_01x04 (DS18B E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, J17 Screw_Terminal_01x04 (Seatalk), J2 Screw_Terminal_01x04 (SHT3X), J4 Screw_Terminal_01x06 (ABX0010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, J6 Conn_01x10_Socket (ADS1115 1), J7 ESP32-S3-N16R8-DevKit_01x22_S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, J9 Screw_Terminal_01x02 (12V Boa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, Q1 BC337, U1 PC817, U2 R-78K5.0-1.0

Commit message: Bring the silkscreen designators back onto the board
J14, J15 and J16 had their reference text centred 0.04 mm past the right
edge, so roughly half of each was cut off - on the three probe terminals
that have to be told apart when the cables go on. J2, J4, J12 and R22 sat
on top of other silkscreen and were no easier to read.

The IMU legend said ABC00101. The part is ABX00101, which is what the
schematic and A-009 have always carried.

Nothing else moved: eight reference field positions and one string. No
track, pad or net is touched, so the exported netlist still describes this
board.

DRC goes from 69 violations to 63. What is left is the courtyard overlap
between C10 and R16, Q1's designator under the fridge probe legend, and
the keep-out rectangles over the ADS1115 sockets, which are deliberate -
the rule that reports them says the silkscreen is clipped at the solder
mask, so the pads stay clear.
Other:
- board text added: "INT SCL SDA GND VIN IMU Modulino ABX00101"
- board text removed: "INT SCL SDA GND VIN IMU Modulino ABC00101"
Changed lines of the file:
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@@
 		(tags "THT terminal block Metz Connect Type101_RT01604HBWC pitch 5.08mm size 20.3x8mm drill 1.3mm pad 2.5mm")
 		(property "Reference" "J16"
-			(at 7.62 -5.12 90)
+			(at -3.81 0 0)
 			(layer "F.SilkS")
 			(effects
@@
 		(tags "THT terminal block Metz Connect Type101_RT01604HBWC pitch 5.08mm size 20.3x8mm drill 1.3mm pad 2.5mm")
 		(property "Reference" "J14"
-			(at 7.62 -5.12 90)
+			(at -3.81 0 0)
 			(layer "F.SilkS")
 			(effects
@@
 		(tags "Resistor Axial_DIN0309 series Axial Horizontal pin pitch 12.7mm 0.5W = 1/2W length 9mm diameter 3.2mm")
 		(property "Reference" "R22"
-			(at 6.35 -2.72 0)
+			(at 6.35 0 0)
 			(layer "F.SilkS")
 			(effects
@@
 		(tags "THT terminal block Metz Connect Type101_RT01604HBWC pitch 5.08mm size 20.3x8mm drill 1.3mm pad 2.5mm")
 		(property "Reference" "J15"
-			(at 7.62 -5.12 90)
+			(at -3.81 0 0)
 			(layer "F.SilkS")
 			(effects
@@
 		(tags "THT terminal block Metz Connect Type101_RT01606HBWC pitch 5.08mm size 30.5x8mm drill 1.3mm pad 2.5mm")
 		(property "Reference" "J4"
-			(at 12.7 -5.12 90)
+			(at -3.81 -1.27 0)
 			(layer "F.SilkS")
 			(effects
@@
 		(tags "THT terminal block Metz Connect Type101_RT01604HBWC pitch 5.08mm size 20.3x8mm drill 1.3mm pad 2.5mm")
 		(property "Reference" "J2"
-			(at 7.62 -5.12 270)
+			(at -3.81 -1.27 180)
 			(layer "F.SilkS")
 			(effects
@@
 		(tags "THT terminal block Metz Connect Type101_RT01602HBWC pitch 5.08mm size 10.2x8mm drill 1.3mm pad 2.5mm")
 		(property "Reference" "J12"
-			(at 2.54 -5.12 0)
+			(at 8.89 0 90)
 			(layer "F.SilkS")
 			(effects
@@
 		)
 	)
-	(gr_text "INT SCL SDA GND VIN\nIMU Modulino ABC00101"
+	(gr_text "INT SCL SDA GND VIN\nIMU Modulino ABX00101"
 		(at 71.12 105.41 90)
 		(layer "F.SilkS")
